Commit message: urdf update, proto broken only base_link

File: src/ros381_description/urdf/ros381.urdf (robot description, URDF)
Before this commit: robot ros381, 2 links, 1 joints
Links:
- added link wheel_left; visual cylinder length=0.039 radius=0.035
- added link wheel_right; visual cylinder length=0.039 radius=0.035
Joints:
- added joint wheel_left: type continuous, parent base_link, child wheel_left, origin xyz=0.0 0.07725 0.035 rpy=1.570796327 0 0, axis 0.0 0.0 -1.0
- added joint wheel_right: type continuous, parent base_link, child wheel_right, origin xyz=0.0 -0.07725 0.035 rpy=1.570796327 0 0, axis 0.0 0.0 -1.0

Commit message: updated urdf with inertial, proto works
also edited colors in proto, they will get overwritten when running
urdf2webots

File: src/ros381_description/urdf/ros381.urdf (robot description, URDF)
Before this commit: robot ros381, 4 links, 3 joints
Links:
- link base_link: mass None -> 2.0
- link bottom_plate: mass None -> 6.0
- link wheel_left: mass None -> 0.1
- link wheel_right: mass None -> 0.1

Commit message: vrte se tockovi, proklizavaju
TODO: povecaj trenje

File: src/ros381_description/urdf/ros381.urdf (robot description, URDF)
Before this commit: robot ros381, 4 links, 3 joints
Links:
- link base_link: geometry collision box size=0.125 0.4 0.325; visual box size=0.125 0.4 0.325
- link bottom_plate: geometry collision box size=0.25 0.4 0.01; visual box size=0.25 0.4 0.01
- link wheel_left: geometry collision cylinder length=0.039 radius=0.035; visual cylinder length=0.039 radius=0.035
- link wheel_right: geometry collision cylinder length=0.039 radius=0.035; visual cylinder length=0.039 radius=0.035

Commit message: odometry blocks (sliders) in urdf

File: src/ros381_description/urdf/ros381.urdf (robot description, URDF)
Before this commit: robot ros381, 4 links, 3 joints
Links:
- added link left_odometry_block; visual box size=0.09 0.015 0.05
- added link right_odometry_block; visual box size=0.09 0.015 0.05
Joints:
- added joint left_odometry_slider: type prismatic, parent base_link, child left_odometry_block, origin xyz=0 0.1485 0.015, axis 0 0 1, limit lower=0.0 upper=0.02 effort=0 velocity=100
- added joint right_odometry_slider: type prismatic, parent base_link, child right_odometry_block, origin xyz=0 -0.1485 0.015, axis 0 0 1, limit lower=0.0 upper=0.02 effort=0 velocity=100

Commit message: update urdf, pozicije odometrijskih blokova

File: src/ros381_description/urdf/ros381.urdf (robot description, URDF)
Before this commit: robot ros381, 6 links, 5 joints
Joints:
- joint left_odometry_slider: origin xyz=0 0.1485 0.015 -> xyz=0 0.134 0.015
- joint right_odometry_slider: origin xyz=0 -0.1485 0.015 -> xyz=0 -0.134 0.015

Commit message: urdf odometry seems great

File: src/ros381_description/urdf/ros381.urdf (robot description, URDF)
Before this commit: robot ros381, 6 links, 5 joints
Links:
- added link odometry_wheel_left, mass 0.055; collision cylinder length=0.002 radius=0.036; visual cylinder length=0.002 radius=0.036
- added link odometry_wheel_right, mass 0.055; collision cylinder length=0.002 radius=0.036; visual cylinder length=0.002 radius=0.036
- link left_odometry_block: mass None -> 0.0622; geometry collision box size=0.09 0.015 0.05; visual box size=0.09 0.015 0.05
- link right_odometry_block: mass None -> 0.0622; geometry collision box size=0.09 0.015 0.05; visual box size=0.09 0.015 0.05
Joints:
- added joint odometry_wheel_left: type continuous, parent left_odometry_block, child odometry_wheel_left, origin xyz=0 0.0145 0 rpy=1.570796327 0 0, axis 0.0 0.0 -1.0
- added joint odometry_wheel_right: type continuous, parent right_odometry_block, child odometry_wheel_right, origin xyz=0 -0.0145 0 rpy=1.570796327 0 0, axis 0.0 0.0 -1.0
- joint left_odometry_slider: limit lower=0.0 upper=0.02 effort=0 velocity=100 -> lower=0.0 upper=0.03 effort=0 velocity=100
- joint right_odometry_slider: limit lower=0.0 upper=0.02 effort=0 velocity=100 -> lower=0.0 upper=0.03 effort=0 velocity=100

Commit message: base.stl in urdf

File: src/ros381_description/urdf/ros381.urdf (robot description, URDF)
Before this commit: robot ros381, 8 links, 7 joints
Links:
- removed link bottom_plate
- link base_link: geometry collision mesh filename=package://ros381_description/meshes/base.stl; visual mesh filename=package://ros381_description/meshes/base.stl
Joints:
- removed joint bottom_plate_to_base
- joint wheel_left: origin xyz=0.0 0.07725 0.035 rpy=1.570796327 0 0 -> xyz=0.0 0.07725 0.032 rpy=1.570796327 0 0
- joint wheel_right: origin xyz=0.0 -0.07725 0.035 rpy=1.570796327 0 0 -> xyz=0.0 -0.07725 0.032 rpy=1.570796327 0 0

Commit message: proto visual mesh, collision cylinder

File: src/ros381_description/urdf/ros381.urdf (robot description, URDF)
Before this commit: robot ros381, 7 links, 6 joints
Links:
- link base_link: geometry collision cylinder length=0.325 radius=0.16; visual mesh filename=package://ros381_description/meshes/base.stl

Commit message: pokusaj collision.stl

File: src/ros381_description/urdf/ros381.urdf (robot description, URDF)
Before this commit: robot ros381, 7 links, 6 joints
Links:
- link base_link: geometry collision mesh filename=package://ros381_description/meshes/base_collision.stl; visual mesh filename=package://ros381_description/meshes/base.stl

Commit message: proto kinda broken

File: src/ros381_description/urdf/ros381.urdf (robot description, URDF)
Before this commit: robot ros381, 7 links, 6 joints
Links:
- added link armor, mass 2.0; collision cylinder length=0.01 radius=0.01; visual mesh filename=package://ros381_description/meshes/armor.stl
Joints:
- added joint armor_joint: type fixed, parent base_link, child armor

Commit message: update collision

File: src/ros381_description/urdf/ros381.urdf (robot description, URDF)
Before this commit: robot ros381, 8 links, 7 joints
Links:
- link armor: geometry collision mesh filename=package://ros381_description/meshes/base_collision.stl; visual mesh filename=package://ros381_description/meshes/armor.stl
- link base_link: geometry collision box size=0.268 0.126 0.002; visual mesh filename=package://ros381_description/meshes/base.stl
Joints:
- joint armor_joint: origin (none) -> xyz=0 0 0 rpy=0 0 1.570796327

Commit message: control improved

File: src/ros381_description/urdf/ros381.urdf (robot description, URDF)
Before this commit: robot ros381, 8 links, 7 joints
Links:
- link base_link: geometry collision cylinder length=0.004 radius=0.14; visual mesh filename=package://ros381_description/meshes/base.stl
