Commit message: lidar proto and urdf

File: src/ros381_description/urdf/blue.urdf (robot description, URDF)
Before this commit: robot blue, 8 links, 7 joints
Links:
- added link lidar, mass 0.1; collision cylinder length=0.08 radius=0.05; visual cylinder length=0.08 radius=0.05
Joints:
- added joint lidar_joint: type fixed, parent base_link, child lidar, origin xyz=0 0 0.376 rpy=0 0 0

File: src/ros381_description/urdf/ros381.urdf (robot description, URDF)
Before this commit: robot ros381, 8 links, 7 joints
Links:
- added link lidar, mass 0.1; collision cylinder length=0.08 radius=0.05; visual cylinder length=0.08 radius=0.05
Joints:
- added joint lidar_joint: type fixed, parent base_link, child lidar, origin xyz=0 0 0.376 rpy=0 0 0

File: src/ros381_description/urdf/yellow.urdf (robot description, URDF)
Before this commit: robot yellow, 8 links, 7 joints
Links:
- added link lidar, mass 0.1; collision cylinder length=0.08 radius=0.05; visual cylinder length=0.08 radius=0.05
Joints:
- added joint lidar_joint: type fixed, parent base_link, child lidar, origin xyz=0 0 0.376 rpy=0 0 0

Commit message: updated protos

File: src/ros381_description/urdf/blue.urdf (robot description, URDF)
Before this commit: robot blue, 9 links, 8 joints
Links:
- link base_link: geometry collision box size=0.125 0.21 0.004; visual mesh filename=package://ros381_description/meshes/base.stl

File: src/ros381_description/urdf/ros381.urdf (robot description, URDF)
Before this commit: robot ros381, 9 links, 8 joints
Links:
- link base_link: geometry collision box size=0.125 0.21 0.004; visual mesh filename=package://ros381_description/meshes/base.stl

File: src/ros381_description/urdf/yellow.urdf (robot description, URDF)
Before this commit: robot yellow, 9 links, 8 joints
Links:
- link base_link: geometry collision box size=0.125 0.21 0.004; visual mesh filename=package://ros381_description/meshes/base.stl
